File: motordriverv2.kicad_sch (KiCad schematic)
At the start: 0 parts

Commit message: pcb geçiş
Other:
- sheet mcu ports: added FET_CAO, FET_FAULT, FET_H_A, FET_H_B, FET_H_C, FET_L_A, FET_L_B, FET_L_C; removed none
Changed lines of the file:
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@@
 	(generator_version "10.0")
 	(paper "A4")
+	(wire
+		(pts
+			(xy 182.88 73.66) (xy 199.39 73.66)
+		)
+		(stroke
+			(width 0)
+			(type default)
+		)
+	)
+	(wire
+		(pts
+			(xy 182.88 76.2) (xy 199.39 76.2)
+		)
+		(stroke
+			(width 0)
+			(type default)
+		)
+	)
+	(wire
+		(pts
+			(xy 182.88 55.88) (xy 199.39 55.88)
+		)
+		(stroke
+			(width 0)
+			(type default)
+		)
+	)
+	(wire
+		(pts
+			(xy 182.88 59.69) (xy 199.39 59.69)
+		)
+		(stroke
+			(width 0)
+			(type default)
+		)
+	)
+	(wire
+		(pts
+			(xy 182.88 64.77) (xy 199.39 64.77)
+		)
+		(stroke
+			(width 0)
+			(type default)
+		)
+	)
+	(wire
+		(pts
+			(xy 182.88 62.23) (xy 199.39 62.23)
+		)
+		(stroke
+			(width 0)
+			(type default)
+		)
+	)
+	(wire
+		(pts
+			(xy 182.88 71.12) (xy 199.39 71.12)
+		)
+		(stroke
+			(width 0)
+			(type default)
+		)
+	)
+	(wire
+		(pts
+			(xy 182.88 52.07) (xy 199.39 52.07)
+		)
+		(stroke
+			(width 0)
+			(type default)
+		)
+	)
 	(sheet
 		(at 149.86 20.32)
@@
 	)
 	(sheet
-		(at 204.47 48.26)
+		(at 199.39 48.26)
 		(size 46.99 59.69)
 		(exclude_from_sim no)
@@
 		)
 		(property "Sheetname" "FET_DRIVER"
-			(at 204.47 47.5484 0)
+			(at 199.39 47.5484 0)
 			(show_name no)
 			(do_not_autoplace no)
@@
 		)
 		(property "Sheetfile" "fet_driver.kicad_sch"
-			(at 204.47 108.5346 0)
+			(at 199.39 108.5346 0)
 			(show_name no)
 			(do_not_autoplace no)
@@
 		)
 		(pin "CA0" input
-			(at 204.47 52.07 180)
+			(at 199.39 52.07 180)
 			(effects
 				(font
@@
 		)
 		(pin "LIN3" input
-			(at 204.47 76.2 180)
+			(at 199.39 76.2 180)
 			(effects
 				(font
@@
 		)
 		(pin "LIN2" input
-			(at 204.47 73.66 180)
+			(at 199.39 73.66 180)
 			(effects
 				(font
@@
 		)
 		(pin "LIN1" input
-			(at 204.47 71.12 180)
+			(at 199.39 71.12 180)
 			(effects
 				(font
@@
 		)
 		(pin "HIN2" input
-			(at 204.47 62.23 180)
+			(at 199.39 62.23 180)
 			(effects
 				(font
@@
 		)
 		(pin "HIN3" input
-			(at 204.47 64.77 180)
+			(at 199.39 64.77 180)
 			(effects
 				(font
@@
 		)
 		(pin "FAULT" input
-			(at 204.47 55.88 180)
+			(at 199.39 55.88 180)
 			(effects
 				(font
@@
 		)
 		(pin "HIN1" input
-			(at 204.47 59.69 180)
+			(at 199.39 59.69 180)
 			(effects
 				(font
@@
 			)
 		)
+		(pin "FET_CAO" input
+			(at 182.88 52.07 0)
+			(effects
+				(font
+					(size 1.27 1.27)
+				)
+				(justify right)
+			)
+		)
+		(pin "FET_FAULT" input
+			(at 182.88 55.88 0)
+			(effects
+				(font
+					(size 1.27 1.27)
+				)
+				(justify right)
+			)
+		)
+		(pin "FET_H_A" output
+			(at 182.88 59.69 0)
+			(effects
+				(font
+					(size 1.27 1.27)
+				)
+				(justify right)
+			)
+		)
+		(pin "FET_H_B" output
+			(at 182.88 62.23 0)
+			(effects
+				(font
+					(size 1.27 1.27)
+				)
+				(justify right)
+			)
+		)
+		(pin "FET_H_C" output
+			(at 182.88 64.77 0)
+			(effects
+				(font
+					(size 1.27 1.27)
+				)
+				(justify right)
+			)
+		)
+		(pin "FET_L_A" output
+			(at 182.88 71.12 0)
+			(effects
+				(font
+					(size 1.27 1.27)
+				)
+				(justify right)
+			)
+		)
+		(pin "FET_L_B" output
+			(at 182.88 73.66 0)
+			(effects
+				(font
+					(size 1.27 1.27)
+				)
+				(justify right)
+			)
+		)
+		(pin "FET_L_C" output
+			(at 182.88 76.2 0)
+			(effects
+				(font
+					(size 1.27 1.27)
+				)
+				(justify right)
+			)
+		)
