File: mcu.kicad_sch (KiCad schematic)
At the start: 35 parts, among them J10 Conn_01x05, J11 Conn_01x05, J15 Conn_01x04, J5 Conn_01x02, J6 Conn_01x02, J7 Conn_01x03, J8 Conn_01x03, J9 HALL INPUT, U8 STM32G474VETx, Y1 8MHz

Commit message: fet tamam
Parts:
- added C37, C38, C39, C40, C41: 100nF, symbol Device:C
- added J16: Conn_01x02, symbol Connector_Generic:Conn_01x02
- added R39, R40, R41, R42, R43, R44: 10K, symbol Device:R
Connections:
- net +3V3: now also J7.3 (Pin_3), J8.3 (Pin_3)
- net GND: now also J5.2 (Pin_2), J6.2 (Pin_2), J7.1 (Pin_1), J8.1 (Pin_1), C37.1, C38.1, C39.1, C40.1, C41.1, J16.2 (Pin_2), R39.2
- net at J6.1 (Pin_1): now also R43.1
- net at U8.33 (PB1): now also R40.1
- net Brake Lights: now reaches U8.34 (PB2)
- net Brake Lights: now also C41.2, R44.2
- net HALT: now reaches U8.38 (PE7)
- net HALT: now also C40.2, R43.2
- net GPIO_BRAKE: now reaches U8.39 (PE8)
- net GPIO_BRAKE: now also C39.2, R42.2
- net at U8.40 (PE9): now also R41.1
- net at J15.2 (Pin_2), R38.2: no longer U8.94 (PB7)
- net at J15.3 (Pin_3), R37.1: no longer U8.95 (PB8)
- net ADC3_Regen: now reaches J7.2 (Pin_2)
- net ADC3_Regen: now also C38.2, R41.2
- net ADC3_ACCELERATOR: now reaches J8.2 (Pin_2)
- net ADC3_ACCELERATOR: now also C37.2, R40.2
- net at J5.1 (Pin_1): now also R42.1
- new net: R39.1, U8.95 (PB8)
- new net: J16.1 (Pin_1), R44.1
- no-connect marks 0 -> 7
Other:
- moved on the sheet: J5, J7

Commit message: pcb geçiş
Parts:
- removed C37: 100nF, symbol Device:C
- removed R40: 10K, symbol Device:R
- added C35: 100nF, Capacitor_SMD:C_0805_2012Metric_Pad1.18x1.45mm_HandSolder, symbol Device:C
- added J10: USB_C_Receptacle_USB2.0_16P, Connector_USB:USB_C_Receptacle_GCT_USB4105-xx-A_16P_TopMnt_Horizontal, symbol Connector:USB_C_Receptacle_USB2.0_16P
- added R12: 10K, Resistor_SMD:R_1210_3225Metric, symbol Device:R
- added U8: TJA1051T, Package_SO:SOIC-8_3.9x4.9mm_P1.27mm, symbol Interface_CAN_LIN:TJA1051T
- C15: renamed from C38; footprint (none) -> Capacitor_SMD:C_0805_2012Metric_Pad1.18x1.45mm_HandSolder
- C16: renamed from C39; footprint (none) -> Capacitor_SMD:C_0805_2012Metric_Pad1.18x1.45mm_HandSolder
- C17: renamed from C40; footprint (none) -> Capacitor_SMD:C_0805_2012Metric_Pad1.18x1.45mm_HandSolder
- C18: renamed from C41; footprint (none) -> Capacitor_SMD:C_0805_2012Metric_Pad1.18x1.45mm_HandSolder
- C19: renamed from C18; footprint Capacitor_SMD:C_1210_3225Metric_Pad1.33x2.70mm_HandSolder -> Capacitor_SMD:C_0603_1608Metric_Pad1.08x0.95mm_HandSolder
- C20: renamed from C19; footprint Capacitor_SMD:C_1210_3225Metric_Pad1.33x2.70mm_HandSolder -> Capacitor_SMD:C_0603_1608Metric_Pad1.08x0.95mm_HandSolder
- C25: renamed from C21; footprint Capacitor_SMD:C_1210_3225Metric_Pad1.33x2.70mm_HandSolder -> Capacitor_SMD:C_0805_2012Metric_Pad1.18x1.45mm_HandSolder
- C26: renamed from C22; footprint Capacitor_SMD:C_1210_3225Metric_Pad1.33x2.70mm_HandSolder -> Capacitor_SMD:C_0805_2012Metric_Pad1.18x1.45mm_HandSolder
- C27: renamed from C23; footprint Capacitor_SMD:C_1210_3225Metric_Pad1.33x2.70mm_HandSolder -> Capacitor_SMD:C_0805_2012Metric_Pad1.18x1.45mm_HandSolder
- C28: renamed from C24; footprint Capacitor_SMD:C_1210_3225Metric_Pad1.33x2.70mm_HandSolder -> Capacitor_SMD:C_0805_2012Metric_Pad1.18x1.45mm_HandSolder
- C29: renamed from C25; footprint Capacitor_SMD:C_1210_3225Metric_Pad1.33x2.70mm_HandSolder -> Capacitor_SMD:C_0805_2012Metric_Pad1.18x1.45mm_HandSolder
- C30: renamed from C26; footprint Capacitor_SMD:C_1210_3225Metric_Pad1.33x2.70mm_HandSolder -> Capacitor_SMD:C_0805_2012Metric_Pad1.18x1.45mm_HandSolder
- C31: renamed from C27; footprint Capacitor_SMD:C_1210_3225Metric_Pad1.33x2.70mm_HandSolder -> Capacitor_SMD:C_0805_2012Metric_Pad1.18x1.45mm_HandSolder
- C32: renamed from C28; footprint Capacitor_SMD:C_1210_3225Metric_Pad1.33x2.70mm_HandSolder -> Capacitor_SMD:C_0805_2012Metric_Pad1.18x1.45mm_HandSolder
- C33: renamed from C29; footprint Capacitor_SMD:C_1210_3225Metric_Pad1.33x2.70mm_HandSolder -> Capacitor_SMD:C_0805_2012Metric_Pad1.18x1.45mm_HandSolder
- C34: renamed from C30; footprint Capacitor_SMD:C_1210_3225Metric_Pad1.33x2.70mm_HandSolder -> Capacitor_SMD:C_0805_2012Metric_Pad1.18x1.45mm_HandSolder
- J11: renamed from J10; footprint (none) -> TerminalBlock_RND:TerminalBlock_RND_205-00004_1x05_P5.00mm_Horizontal
- J13: renamed from J15; footprint (none) -> TerminalBlock_RND:TerminalBlock_RND_205-00003_1x04_P5.00mm_Horizontal
- J14: renamed from J11; footprint (none) -> TerminalBlock_RND:TerminalBlock_RND_205-00004_1x05_P5.00mm_Horizontal
- J5: renamed from J8; footprint (none) -> TerminalBlock_RND:TerminalBlock_RND_205-00002_1x03_P5.00mm_Horizontal
- J6: renamed from J7; footprint (none) -> TerminalBlock_RND:TerminalBlock_RND_205-00002_1x03_P5.00mm_Horizontal
- J7: renamed from J5; footprint (none) -> TerminalBlock_RND:TerminalBlock_RND_205-00001_1x02_P5.00mm_Horizontal
- J8: renamed from J6; footprint (none) -> TerminalBlock_RND:TerminalBlock_RND_205-00001_1x02_P5.00mm_Horizontal
- J9: renamed from J16; footprint (none) -> TerminalBlock_RND:TerminalBlock_RND_205-00001_1x02_P5.00mm_Horizontal
- R1: renamed from R41; footprint (none) -> Resistor_SMD:R_1210_3225Metric
- R11: renamed from R39; footprint (none) -> Resistor_SMD:R_1210_3225Metric
- R13: renamed from R38; footprint (none) -> Resistor_SMD:R_1210_3225Metric
- R14: renamed from R37; footprint (none) -> Resistor_SMD:R_1210_3225Metric
- R15: renamed from R7; footprint (none) -> Resistor_SMD:R_1210_3225Metric
- R2: renamed from R42; footprint (none) -> Resistor_SMD:R_1210_3225Metric
- R3: renamed from R43; footprint (none) -> Resistor_SMD:R_1210_3225Metric
- R4: renamed from R44; footprint (none) -> Resistor_SMD:R_1210_3225Metric
- Y1: footprint (none) -> Crystal:Crystal_HC18-U_Vertical
- renumbered C15 to C21, C16 to C22, C17 to C23, C20 to C24, J9 to J12, R6 to R10, R1 to R5, R2 to R6, R3 to R7, R4 to R8, R5 to R9, U8 to U9
Connections:
- net ADC3_ACCELERATOR: now also U9.33 (PB1), C35.2, R12.2; no longer J5.2 (Pin_2)
- net ADC3_Regen: now also R1.1, U9.40 (PE9); no longer C15.2, J6.2 (Pin_2), R1.2
- net FET_H_A: now also U9.71 (PA10); no longer U9.69 (PA8)
- net FET_H_B: now also U9.69 (PA8); no longer U9.71 (PA10)
- net FET_L_A: now also U9.72 (PA11); no longer U9.70 (PA9)
- net FET_L_B: now also U9.70 (PA9); no longer U9.72 (PA11)
- net GND: now also C35.1, J10.A1 (GND), J10.A12 (GND), J10.B1 (GND), J10.B12 (GND), J10.SH (SHIELD), U8.2 (GND), U8.8 (S)
- net at U9.65 (PC6): now also J13.2 (Pin_2), R13.2
- net at U9.66 (PC7): now also J13.3 (Pin_3), R14.1
- net CAN_RX: now reaches U9.82 (PD0)
- net CAN_RX: now also U8.1 (TXD)
- net CAN_TX: now reaches U9.83 (PD1)
- new net: J10.A7 (D-), J10.B7 (D-), U8.6 (CANL)
- new net: J10.A6 (D+), J10.B6 (D+), U8.7 (CANH)
- new net: J10.A4 (VBUS), J10.A9 (VBUS), J10.B4 (VBUS), J10.B9 (VBUS)
- new net: C15.2, J6.2 (Pin_2), R1.2
- new net: J5.2 (Pin_2), R12.1
- no-connect marks 7 -> 60
Other:
- moved on the sheet: C15, C16, C17, C18, C19, C20, C21, C22, C23, C24, C25, C26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

Commit message: pcb geçiş v2
Parts:
- added R33: 10k, Resistor_SMD:R_0805_2012Metric_Pad1.20x1.40mm_HandSolder, symbol Device:R
- J14: footprint TerminalBlock_RND:TerminalBlock_RND_205-00004_1x05_P5.00mm_Horizontal -> Connector_PinSocket_2.54mm:PinSocket_1x05_P2.54mm_Vertical
- R1, R11, R12, R13, R14, R15, R2, R3, R4: footprint Resistor_SMD:R_1210_3225Metric -> Resistor_SMD:R_0805_2012Metric_Pad1.20x1.40mm_HandSolder
Connections:
- net +3V3: now also R33.1
- net ADC3_Regen: now also C15.2
- net NRST: now also R33.2
- net at J6.2 (Pin_2), R1.2: no longer C15.2
Other:
- moved on the sheet: R1
Changed lines of the file:
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@@
 	)
 	(junction
-		(at 266.7 82.55)
+		(at 270.51 106.68)
 		(diameter 0)
 		(color 0 0 0 0)
 	)
 	(junction
-		(at 270.51 106.68)
+		(at 248.92 20.32)
 		(diameter 0)
 		(color 0 0 0 0)
 	)
 	(junction
-		(at 248.92 20.32)
+		(at 90.17 41.91)
 		(diameter 0)
 		(color 0 0 0 0)
 	)
 	(junction
-		(at 90.17 41.91)
+		(at 266.7 82.55)
 		(diameter 0)
 		(color 0 0 0 0)
@@
 	)
 	(junction
+		(at 49.53 69.85)
+		(diameter 0)
+		(color 0 0 0 0)
+	)
+	(junction
 		(at 87.63 34.29)
 		(diameter 0)
@@
 	(wire
 		(pts
+			(xy 46.99 69.85) (xy 49.53 69.85)
+		)
+		(stroke
+			(width 0)
+			(type default)
+		)
+	)
+	(wire
+		(pts
 			(xy 110.49 162.56) (xy 137.16 162.56)
 		)
@@
 	(wire
 		(pts
-			(xy 246.38 82.55) (xy 266.7 82.55)
+			(xy 246.38 82.55) (xy 259.08 82.55)
 		)
 		(stroke
@@
 	(wire
 		(pts
+			(xy 266.7 82.55) (xy 274.32 82.55)
+		)
+		(stroke
+			(width 0)
+			(type default)
+		)
+	)
+	(wire
+		(pts
 			(xy 264.16 101.6) (xy 264.16 104.14)
 		)
@@
 	)
 	(label "NRST"
-		(at 49.53 69.85 180)
+		(at 46.99 69.85 180)
 		(effects
 			(font
@@
 			)
 		)
-		(property "Footprint" "Resistor_SMD:R_1210_3225Metric"
+		(property "Footprint" "Resistor_SMD:R_0805_2012Metric_Pad1.20x1.40mm_HandSolder"
 			(at 266.7 108.458 90)
 			(hide yes)
@@
 			)
 		)
-		(property "Footprint" "Resistor_SMD:R_1210_3225Metric"
+		(property "Footprint" "Resistor_SMD:R_0805_2012Metric_Pad1.20x1.40mm_HandSolder"
 			(at 140.462 83.82 90)
 			(hide yes)
@@
 			)
 		)
-		(property "Footprint" "Resistor_SMD:R_1210_3225Metric"
+		(property "Footprint" "Resistor_SMD:R_0805_2012Metric_Pad1.20x1.40mm_HandSolder"
 			(at 124.46 123.698 90)
 			(hide yes)
@@
 	)
 	(symbol
+		(lib_id "power:+3V3")
+		(at 49.53 62.23 0)
+		(unit 1)
+		(body_style 1)
+		(exclude_from_sim no)
+		(in_bom yes)
+		(on_board yes)
+		(in_pos_files yes)
+		(dnp no)
+		(fields_autoplaced yes)
+		(property "Reference" "#PWR012"
+			(at 49.53 66.04 0)
+			(hide yes)
+			(show_name no)
+			(do_not_autoplace no)
+			(effects
+				(font
+					(size 1.27 1.27)
+				)
+			)
+		)
+		(property "Value" "+3V3"
+			(at 49.53 57.15 0)
+			(show_name no)
+			(do_not_autoplace no)
+			(effects
+				(font
+					(size 1.27 1.27)
+				)
+			)
+		)
+		(property "Footprint" ""
+			(at 49.53 62.23 0)
+			(hide yes)
+			(show_name no)
+			(do_not_autoplace no)
+			(effects
+				(font
+					(size 1.27 1.27)
+				)
+			)
+		)
+		(property "Datasheet" ""
+			(at 49.53 62.23 0)
+			(hide yes)
+			(show_name no)
+			(do_not_autoplace no)
+			(effects
+				(font
+					(size 1.27 1.27)
+				)
+			)
+		)
+		(property "Description" "Power symbol creates a global label with name \"+3V3\""
+			(at 49.53 62.23 0)
+			(hide yes)
+			(show_name no)
+			(do_not_autoplace no)
+			(effects
+				(font
+					(size 1.27 1.27)
+				)
+			)
+		)
+		(pin "1"
+		)
+		(instances
+			(project "motordriverv2"
+				(path "/a575d6d2-ca2d-48e8-a0bf-4cf8349556d4/3f98f0ea-9852-4672-9467-6a0340feaa03"
+					(reference "#PWR012")
+					(unit 1)
+				)
+			)
+		)
+	)
+	(symbol
 		(lib_id "Device:C")
 		(at 203.2 -12.7 90)
@@
 			)
 		)
-		(property "Footprint" "Resistor_SMD:R_1210_3225Metric"
+		(property "Footprint" "Resistor_SMD:R_0805_2012Metric_Pad1.20x1.40mm_HandSolder"
 			(at 135.382 166.37 90)
 			(hide yes)
@@
 			)
 		)
-		(property "Footprint" "Resistor_SMD:R_1210_3225Metric"
+		(property "Footprint" "Resistor_SMD:R_0805_2012Metric_Pad1.20x1.40mm_HandSolder"
 			(at 266.7 142.748 90)
 			(hide yes)
@@
 	)
 	(symbol
+		(lib_id "Device:R")
+		(at 49.53 66.04 0)
+		(unit 1)
+		(body_style 1)
+		(exclude_from_sim no)
+		(in_bom yes)
+		(on_board yes)
+		(in_pos_files yes)
+		(dnp no)
+		(property "Reference" "R33"
+			(at 52.07 64.7699 0)
+			(show_name no)
+			(do_not_autoplace no)
+			(effects
+				(font
+					(size 1.27 1.27)
+				)
+				(justify left)
+			)
+		)
+		(property "Value" "10k"
+			(at 49.53 67.564 90)
+			(show_name no)
+			(do_not_autoplace no)
+			(effects
+				(font
+					(size 1.27 1.27)
+				)
+				(justify left)
+			)
+		)
+		(property "Footprint" "Resistor_SMD:R_0805_2012Metric_Pad1.20x1.40mm_HandSolder"
+			(at 47.752 66.04 90)
+			(hide yes)
+			(show_name no)
+			(do_not_autoplace no)
+			(effects
+				(font
+					(size 1.27 1.27)
+				)
+			)
+		)
+		(property "Datasheet" ""
+			(at 49.53 66.04 0)
+			(hide yes)
+			(show_name no)
+			(do_not_autoplace no)
+			(effects
+				(font
+					(size 1.27 1.27)
+				)
+			)
+		)
+		(property "Description" "Resistor"
+			(at 49.53 66.04 0)
+			(hide yes)
+			(show_name no)
+			(do_not_autoplace no)
+			(effects
+				(font
+					(size 1.27 1.27)
+				)
+			)
+		)
+		(pin "2"
+		)
+		(pin "1"
+		)
+		(instances
+			(project "motordriverv2"
+				(path "/a575d6d2-ca2d-48e8-a0bf-4cf8349556d4/3f98f0ea-9852-4672-9467-6a0340feaa03"
+					(reference "R33")
+					(unit 1)
+				)
+			)
+		)
+	)
+	(symbol
 		(lib_id "Connector_Generic:Conn_01x05")
 		(at 128.27 69.85 0)
@@
 			)
 		)
-		(property "Footprint" "TerminalBlock_RND:TerminalBlock_RND_205-00004_1x05_P5.00mm_Horizontal"
+		(property "Footprint" "Connector_PinSocket_2.54mm:PinSocket_1x05_P2.54mm_Vertical"
 			(at 242.57 39.37 0)
 			(hide yes)
@@
 			)
 		)
-		(property "Footprint" "Resistor_SMD:R_1210_3225Metric"
+		(property "Footprint" "Resistor_SMD:R_0805_2012Metric_Pad1.20x1.40mm_HandSolder"
 			(at 266.7 124.968 90)
 			(hide yes)
@@
 			)
 		)
-		(property "Footprint" "Resistor_SMD:R_1210_3225Metric"
+		(property "Footprint" "Resistor_SMD:R_0805_2012Metric_Pad1.20x1.40mm_HandSolder"
 			(at 266.7 65.278 90)
 			(hide yes)
@@
 			)
 		)
-		(property "Footprint" "Resistor_SMD:R_1210_3225Metric"
+		(property "Footprint" "Resistor_SMD:R_0805_2012Metric_Pad1.20x1.40mm_HandSolder"
 			(at 135.382 156.21 90)
 			(hide yes)
@@
 	(symbol
 		(lib_id "Device:R")
-		(at 270.51 82.55 270)
+		(at 262.89 82.55 270)
 		(unit 1)
 		(body_style 1)
@@
 		(dnp no)
 		(property "Reference" "R1"
-			(at 269.494 84.582 90)
+			(at 261.874 84.582 90)
 			(show_name no)
 			(do_not_autoplace no)
@@
 		)
 		(property "Value" "10K"
-			(at 268.732 82.55 90)
+			(at 261.112 82.55 90)
 			(show_name no)
 			(do_not_autoplace no)
@@
 			)
 		)
-		(property "Footprint" "Resistor_SMD:R_1210_3225Metric"
-			(at 270.51 80.772 90)
+		(property "Footprint" "Resistor_SMD:R_0805_2012Metric_Pad1.20x1.40mm_HandSolder"
+			(at 262.89 80.772 90)
 			(hide yes)
 			(show_name no)
@@
 		)
 		(property "Datasheet" ""
-			(at 270.51 82.55 0)
+			(at 262.89 82.55 0)
 			(hide yes)
 			(show_name no)
@@
 		)
 		(property "Description" "Resistor"
-			(at 270.51 82.55 0)
+			(at 262.89 82.55 0)
 			(hide yes)
 			(show_name no)

Commit message: pcb geçiş v2
Parts:
- removed J11: Conn_01x05, TerminalBlock_RND:TerminalBlock_RND_205-00004_1x05_P5.00mm_Horizontal, symbol Connector_Generic:Conn_01x05
- added R27: 10K, Resistor_SMD:R_0805_2012Metric_Pad1.20x1.40mm_HandSolder, symbol Device:R
- J13: footprint TerminalBlock_RND:TerminalBlock_RND_205-00003_1x04_P5.00mm_Horizontal -> Connector_PinHeader_2.54mm:PinHeader_1x04_P2.54mm_Vertical
Connections:
- net +5V: now also J10.A4 (VBUS), J10.A9 (VBUS), J10.B4 (VBUS), J10.B9 (VBUS), U8.3 (VCC)
- net CAN_TX: now also U8.4 (RXD)
- net at J10.A7 (D-), J10.B7 (D-), U8.6 (CANL): now also R27.2
- net at J10.A6 (D+), J10.B6 (D+), U8.7 (CANH): now also R27.1
- net MISO: no longer names the net of U9.28 (PA6)
- net MOSI: no longer names the net of U9.29 (PA7)
- net SPICLK: no longer names the net of U9.27 (PA5)
- no-connect marks 60 -> 63
Other:
- moved on the sheet: U8
