File: fet_driver.kicad_sch (KiCad schematic)
At the start: 66 parts, among them J12 PHASE_A, J13 PHASE_B, J14 PHASE_C, Q1 IAUS300N08S5N014TATMA1, Q10 IAUS300N08S5N014TATMA1, Q11 IAUS300N08S5N014TATMA13, Q12 IAUS300N08S5N014TATMA13, Q13 SS8050, Q14 SS8550, Q15 SS8050, Q16 SS8550, Q17 SS8050, Q18 SS8550, Q19 SS8050, Q2 IAUS300N08S5N014TATMA1, Q20 SS8550, Q21 SS8050, Q22 SS8550, Q23 SS8050, Q24 SS8550, Q3 IAUS300N08S5N014TATMA1, Q4 IAUS300N08S5N014TATMA1, Q5 IAUS300N08S5N014TATMA13, Q6 IAUS300N08S5N014TATMA13, Q7 IAUS300N08S5N014TATMA1, Q8 IAUS300N08S5N014TATMA1, Q9 IAUS300N08S5N014TATMA1, U9 IR2130

Commit message: pcb geçiş
Parts:
- removed Q1, Q10, Q2, Q3, Q4, Q7, Q8, Q9: IAUS300N08S5N014TATMA1, IAUS300N08S5N014TATMA1:IAUS300N08S5N014TATMA1, symbol IAUS300N08S5N014ATMA1:IAUS300N08S5N014ATMA1
- removed Q11, Q12, Q6: IAUS300N08S5N014TATMA13, IAUS300N08S5N014TATMA1:IAUS300N08S5N014TATMA1, symbol IAUS300N08S5N014ATMA1:IAUS300N08S5N014ATMA1
- removed R20, R21, R22, R23, R24, R25: 10R, Resistor_SMD:R_1210_3225Metric, symbol Device:R
- removed R26, R27, R28, R29, R30, R31: 10K, Resistor_SMD:R_1210_3225Metric, symbol Device:R
- added Q18, Q19, Q20, Q21, Q22: IAUS300N08S5N014TATMA13, IAUS300N08S5N014TATMA1:IAUS300N08S5N014TATMA1, symbol IAUS300N08S5N014ATMA1:IAUS300N08S5N014ATMA1
- U10: renamed from U9; footprint IR2130:DIP1524W45P254L3740H635Q28 -> Package_DIP:DIP-28_W15.24mm
- renumbered C34 to C36, C35 to C37, C36 to C38, C31 to C39, C32 to C40, C33 to C41, J12 to J15, J13 to J16, J14 to J17, Q13 to Q1, Q22 to Q10, Q23 to Q11, Q24 to Q12, Q5 to Q17, Q14 to Q2, Q15 to Q3, Q16 to Q4, Q17 to Q5, Q18 to Q6, Q19 to Q7, Q20 to Q8, Q21 to Q9, R32 to R16, R33 to R17, R34 to R18, R35 to R19, R36 to R20, R8 to R21, R9 to R22, R10 to R23, R11 to R24, R12 to R25, R13 to R26, R14 to R27, R15 to R28, R16 to R29, R17 to R30, R18 to R31, R19 to R32
Connections:
- net +VDC: now also Q17.10, Q17.11, Q17.12, Q17.13, Q17.14, Q17.15, Q17.16, Q19.10, Q19.11, Q19.12, Q19.13, Q19.14, Q19.15, Q19.16, Q19.9, Q20.10, Q20.11, Q20.12, Q20.13, Q20.14, Q20.15, Q20.16, Q20.9
- net MOS_NEG: now also Q18.1, Q18.2, Q18.3, Q18.4, Q18.5, Q18.6, Q18.7, Q18.8, Q21.1, Q21.2, Q21.3, Q21.4, Q21.5, Q21.6, Q21.7, Q21.8, Q22.1, Q22.2, Q22.3, Q22.4, Q22.5, Q22.6, Q22.7, Q22.8
- net VS1: now also Q19.1, Q19.2, Q19.3, Q19.4, Q19.5, Q19.6, Q19.7, Q19.8, Q21.10, Q21.11, Q21.12, Q21.13, Q21.14, Q21.15, Q21.16, Q21.9
- net VS2: now also Q20.1, Q20.2, Q20.3, Q20.4, Q20.5, Q20.6, Q20.7, Q20.8, Q22.10, Q22.11, Q22.12, Q22.13, Q22.14, Q22.15, Q22.16, Q22.9
- net VS3: now also Q17.1, Q18.10, Q18.11, Q18.12, Q18.13, Q18.14, Q18.15, Q18.16, Q18.9
- net at R21.2, R27.1: now also Q22.8
- net at R25.2, R31.1: now also Q17.8; no longer Q17.1
- net at R26.2, R32.1: now also Q18.8
- net at R24.2, R30.2: now also Q20.8
- net at R23.2, R29.1: now also Q21.8
- net at R22.2, R28.2: now also Q19.8
Other:
- moved on the sheet: C36, C37, C38, C39, C40, C41, D1, D2, D3, J15, J16, J17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

Commit message: pcb geçiş v2
Parts:
- R21: footprint Resistor_SMD:R_1210_3225Metric -> Resistor_SMD:R_0805_2012Metric_Pad1.20x1.40mm_HandSolder
Changed lines of the file:
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@@
 			)
 		)
-		(property "Footprint" "Resistor_SMD:R_1210_3225Metric"
+		(property "Footprint" "Resistor_SMD:R_0805_2012Metric_Pad1.20x1.40mm_HandSolder"
 			(at 207.01 112.268 90)
 			(hide yes)

Commit message: pcb geçiş v2
Parts:
- removed C36: 1nF, Capacitor_SMD:C_1210_3225Metric_Pad1.33x2.70mm_HandSolder, symbol Device:C
- removed Q1, Q11, Q3, Q5, Q7, Q9: SS8050, Package_TO_SOT_SMD:SOT-23, symbol Transistor_BJT:SS8050
- removed Q10, Q12, Q2, Q4, Q6, Q8: SS8550, Package_TO_SOT_SMD:SOT-23, symbol Transistor_BJT:SS8550
- removed Q17, Q18: IAUS300N08S5N014TATMA13, IAUS300N08S5N014TATMA1:IAUS300N08S5N014TATMA1, symbol IAUS300N08S5N014ATMA1:IAUS300N08S5N014ATMA1
- removed R27, R28, R29, R30, R31, R32: 10K, Resistor_SMD:R_1210_3225Metric, symbol Device:R
- added C42: 1nF, Capacitor_SMD:C_1210_3225Metric_Pad1.33x2.70mm_HandSolder, symbol Device:C
- added Q23, Q24: IAUS300N08S5N014TATMA13, IAUS300N08S5N014TATMA1:IAUS300N08S5N014TATMA1, symbol IAUS300N08S5N014ATMA1:IAUS300N08S5N014ATMA1
- added U11, U12, U13, U14, U5, U6: TC4422, Package_DIP:DIP-8_W7.62mm, symbol Driver_FET:TC4422
- R16: value 75K -> 22K
- R19: value 1mR -> 10mR; footprint Resistor_SMD:R_1210_3225Metric -> Resistor_SMD:R_Shunt_Vishay_WSR2_WSR3_KelvinConnection; symbol Device:R -> Device:R_Shunt
- R21: footprint Resistor_SMD:R_0805_2012Metric_Pad1.20x1.40mm_HandSolder -> Resistor_SMD:R_1210_3225Metric_Pad1.30x2.65mm_HandSolder
Connections:
- net +12V: now also D1.2 (A), D3.2 (A), U11.1 (VDD), U11.8 (VDD), U12.1 (VDD), U12.8 (VDD), U13.1 (VDD), U13.8 (VDD), U14.1 (VDD), U14.8 (VDD), U5.1 (VDD), U5.8 (VDD), U6.1 (VDD), U6.8 (VDD)
- net +VDC: now also Q23.10, Q23.11, Q23.12, Q23.13, Q23.14, Q23.15, Q23.16, Q23.9
- net -VDC: now also R19.2, C42.1, U11.4 (GND), U11.5 (GND), U12.4 (GND), U12.5 (GND), U13.4 (GND), U13.5 (GND), U14.4 (GND), U14.5 (GND), U5.4 (GND), U5.5 (GND), U6.4 (GND), U6.5 (GND); no longer C37.2, C38.2
- net CA0: now also R16.2
- net HO1: now also U5.6 (OUTPUT), U5.7 (OUTPUT)
- net HO2: now also U6.6 (OUTPUT), U6.7 (OUTPUT)
- net HO3: now also U11.6 (OUTPUT), U11.7 (OUTPUT)
- net LO1: now also U12.6 (OUTPUT), U12.7 (OUTPUT)
- net LO2: now also U13.6 (OUTPUT), U13.7 (OUTPUT)
- net LO3: now also U14.6 (OUTPUT), U14.7 (OUTPUT)
- net MOS_NEG: now also R19.4, Q24.1, Q24.2, Q24.3, Q24.4, Q24.5, Q24.6, Q24.7; no longer Q21.8, Q22.8, R19.2, R20.1, U10.13 (VS0)
- net VS1: no longer Q19.8
- net VS2: no longer Q20.8
- net VS3: now also Q23.1, Q23.2, Q23.3, Q23.4, Q23.5, Q23.6, Q23.7, Q24.10, Q24.11, Q24.12, Q24.13, Q24.14, Q24.15, Q24.16, Q24.9
- net at R25.2: now also Q23.8
- net at R26.2: now also Q24.8
- net at R16.1: now also R17.1, U10.11 (CA-)
- net HOT1: no longer names the net of U10.27 (HO1)
- net HOT1: now also U5.2 (INPUT)
- net HOT2: no longer names the net of U10.23 (HO2)
- net HOT2: now also U6.2 (INPUT)
- net HOT3: no longer names the net of U10.19 (HO3)
- net HOT3: now also U11.2 (INPUT)
- net LOT1: no longer names the net of U10.16 (LO1)
- net LOT1: now also U12.2 (INPUT)
- net LOT2: no longer names the net of U10.15 (LO2)
- net LOT2: now also U13.2 (INPUT)
- net LOT3: no longer names the net of U10.14 (LO3)
- net LOT3: now also U14.2 (INPUT)
- new net: R19.3, R20.1, U10.13 (VS0)
- new net: C37.2, C38.2, C42.2
Other:
- moved on the sheet: R20

Commit message: pcb geçiş v2
Parts:
- added C36, C43, C44, C45, C46, C47: 100nF, symbol Device:C
- added C4, C5: 660uF, symbol Device:C
- added C48, C49, C50: 10uF, Capacitor_SMD:C_1210_3225Metric_Pad1.33x2.70mm_HandSolder, symbol Device:C
- C39, C40, C41: value 2.2uF -> 10uF
Connections:
- net +12V: now also C36.1, C4.1, C43.1, C44.1, C45.1, C46.1, C47.1, C48.1, C49.1, C5.1, C50.1
- net -VDC: now also C36.2, C4.2, C43.2, C44.2, C45.2, C46.2, C47.2, C48.2, C49.2, C5.2, C50.2
Other:
- note added: "Bulking CAPS"
- note added: "C Caps"

Commit message: pcb geçiş v2
Parts:
- added C51, C52, C53: 100nF, Capacitor_SMD:C_1210_3225Metric_Pad1.33x2.70mm_HandSolder, symbol Device:C
- C36, C43, C44, C45, C46, C47: footprint (none) -> Capacitor_SMD:C_1210_3225Metric_Pad1.33x2.70mm_HandSolder
- C4, C5: value 660uF -> 680uF; footprint (none) -> Capacitor_THT:CP_Radial_D10.0mm_P5.00mm
- Q24: footprint IAUS300N08S5N014TATMA1:IAUS300N08S5N014TATMA1 -> IAUS300N08S5N014TATMA1:IAUS300N08S5N014TATMA
Connections:
- net +12V: now also C51.1, C52.1, C53.1
- net -VDC: now also C51.2, C52.2, C53.2; no longer C4.2, C5.2
- new net GND: C4.2, C5.2
