File: power_IN.kicad_sch (KiCad schematic)
At the start: 26 parts, among them J1 Conn_01x02, J2 PHASE_A, J3 PHASE_A, J4 58-8 OUTPUT, U1 LM2931-5.0_TO220, U2 XC6206PxxxMR, U3 XC6206PxxxMR, U4 LM2931-5.0_TO220, U5 XC6206PxxxMR, U6 XC6206PxxxMR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

Commit message: fet tamam
Parts:
- J2: value PHASE_A -> +VDC
- J3: value PHASE_A -> -VDC
Changed lines of the file:
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@@
 			)
 		)
-		(property "Value" "PHASE_A"
+		(property "Value" "-VDC"
 			(at 239.395 127 0)
 			(show_name no)
@@
 			)
 		)
-		(property "Value" "PHASE_A"
+		(property "Value" "+VDC"
 			(at 239.395 115.57 0)
 			(show_name no)

Commit message: pcb geçiş
Parts:
- removed C11, C12, C8, C9: 100nF, Capacitor_SMD:C_1210_3225Metric_Pad1.33x2.70mm_HandSolder, symbol Device:C
- removed U5, U6: XC6206PxxxMR, Package_TO_SOT_SMD:SOT-23-3, symbol Regulator_Linear:XC6206PxxxMR
- J1: footprint (none) -> TerminalBlock_RND:TerminalBlock_RND_205-00001_1x02_P5.00mm_Horizontal
- J4: footprint (none) -> TerminalBlock_Ningbo-Kagnex:TerminalBlock_Ningbo-Kagnex_HB9500_1x02_P9.5mm
- NT1: footprint (none) -> NetTie:NetTie-2_SMD_Pad2.0mm
- U1, U4, U7: value LM2931-5.0_TO220 -> LM7805
Other:
- moved on the sheet: C1, C10, C13, C14, C2, C3, C4, C5, C6, C7, J1, J2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

Commit message: pcb geçiş v2
Parts:
- removed C10, C4, C5, C7: 100nF, Capacitor_SMD:C_1210_3225Metric_Pad1.33x2.70mm_HandSolder, symbol Device:C
- removed U3: XC6206PxxxMR, Package_TO_SOT_SMD:SOT-23-3, symbol Regulator_Linear:XC6206PxxxMR
- removed U4: LM7805, Package_TO_SOT_THT:TO-220-3_Vertical, symbol Regulator_Linear:LM2931-5.0_TO220
- J4: value 58-8 OUTPUT -> Conn_01x02; footprint TerminalBlock_Ningbo-Kagnex:TerminalBlock_Ningbo-Kagnex_HB9500_1x02_P9.5mm -> TerminalBlock_RND:TerminalBlock_RND_205-00001_1x02_P5.00mm_Horizontal
Other:
- moved on the sheet: C1, C13, C14, C2, C3, C6, J1, J2, J3, NT1, U1, U2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

Commit message: pcb geçiş v2
Parts:
- added C10, C9: 4.7uF, Capacitor_SMD:C_1210_3225Metric_Pad1.33x2.70mm_HandSolder, symbol Device:C
- added C7: 1000uF / 100V, Capacitor_THT:CP_Radial_D18.0mm_P7.50mm, symbol Device:C
- added C8: 1000uF 100V, Capacitor_THT:CP_Radial_D18.0mm_P7.50mm, symbol Device:C
Connections:
- net +VDC: now also C10.1, C7.1, C8.1, C9.1
- net -VDC: now also C10.2, C7.2, C8.2, C9.2
