File: motordriverv2.kicad_pcb (KiCad board)
At the start: 2 copper layers, 20 parts, among them J1 PHASE_B, J2 PHASE_A, J3 PHASE_C, U1 STM32G474VETx, U2 IR2133

Commit message: pcb geçiş
Parts:
- removed R34, R35, R36, R37, R38, R39, R40, R41: 10R, Resistor_SMD:R_1210_3225Metric
- added C1: 100nF, Capacitor_SMD:C_1210_3225Metric_Pad1.33x2.70mm_HandSolder, F.Cu at (485.4, 85.8)
- added C10: 100nF, Capacitor_SMD:C_1210_3225Metric_Pad1.33x2.70mm_HandSolder, F.Cu at (491.4, 102.8)
- added C11: 100nF, Capacitor_SMD:C_1210_3225Metric_Pad1.33x2.70mm_HandSolder, F.Cu at (497.4, 85.8)
- added C12: 100nF, Capacitor_SMD:C_1210_3225Metric_Pad1.33x2.70mm_HandSolder, F.Cu at (497.4, 90.0)
- added C13: 100nF, Capacitor_SMD:C_1210_3225Metric_Pad1.33x2.70mm_HandSolder, F.Cu at (497.4, 94.2)
- added C14: 100nF, Capacitor_SMD:C_1210_3225Metric_Pad1.33x2.70mm_HandSolder, F.Cu at (497.4, 98.5)
- added C15: 100nF, Capacitor_SMD:C_0805_2012Metric_Pad1.18x1.45mm_HandSolder, F.Cu at (92.9, 90.1)
- added C16: 100nF, Capacitor_SMD:C_0805_2012Metric_Pad1.18x1.45mm_HandSolder, F.Cu at (92.9, 93.1)
- added C17: 100nF, Capacitor_SMD:C_0805_2012Metric_Pad1.18x1.45mm_HandSolder, F.Cu at (92.9, 96.1)
- added C18: 100nF, Capacitor_SMD:C_0805_2012Metric_Pad1.18x1.45mm_HandSolder, F.Cu at (92.9, 99.1)
- added C19: 22pF, Capacitor_SMD:C_0603_1608Metric_Pad1.08x0.95mm_HandSolder, F.Cu at (81.3, 63.0)
- added C2: 100nF, Capacitor_SMD:C_1210_3225Metric_Pad1.33x2.70mm_HandSolder, F.Cu at (485.4, 90.0)
- added C20: 22pF, Capacitor_SMD:C_0603_1608Metric_Pad1.08x0.95mm_HandSolder, F.Cu at (81.3, 66.3)
- added C21: 10nF, Capacitor_SMD:C_1210_3225Metric_Pad1.33x2.70mm_HandSolder, F.Cu at (238.6, 54.3)
- added C22: 10nF, Capacitor_SMD:C_1210_3225Metric_Pad1.33x2.70mm_HandSolder, F.Cu at (238.6, 58.6)
- added C23: 10nF, Capacitor_SMD:C_1210_3225Metric_Pad1.33x2.70mm_HandSolder, F.Cu at (238.6, 62.8)
- added C24: 4.7uF, Capacitor_SMD:C_1210_3225Metric_Pad1.33x2.70mm_HandSolder, B.Cu at (80.6, 56.9)
- added C25: 100nF, Capacitor_SMD:C_0805_2012Metric_Pad1.18x1.45mm_HandSolder, B.Cu at (98.4, 64.7)
- added C26: 100nF, Capacitor_SMD:C_0805_2012Metric_Pad1.18x1.45mm_HandSolder, B.Cu at (96.1, 72.8)
- added C27: 100nF, Capacitor_SMD:C_0805_2012Metric_Pad1.18x1.45mm_HandSolder, B.Cu at (98.4, 59.1)
- added C28: 100nF, Capacitor_SMD:C_0805_2012Metric_Pad1.18x1.45mm_HandSolder, B.Cu at (85.0, 57.3)
- added C29: 100nF, Capacitor_SMD:C_0805_2012Metric_Pad1.18x1.45mm_HandSolder, B.Cu at (85.2, 62.5)
- added C3: 100nF, Capacitor_SMD:C_1210_3225Metric_Pad1.33x2.70mm_HandSolder, B.Cu at (86.4, 51.6)
- added C30: 100nF, Capacitor_SMD:C_0805_2012Metric_Pad1.18x1.45mm_HandSolder, B.Cu at (83.0, 70.2)
- added C31: 1uF, Capacitor_SMD:C_0805_2012Metric_Pad1.18x1.45mm_HandSolder, B.Cu at (88.1, 73.7)
- added C32: 10nF, Capacitor_SMD:C_0805_2012Metric_Pad1.18x1.45mm_HandSolder, B.Cu at (88.1, 71.7)
- added C33: 100nF, Capacitor_SMD:C_0805_2012Metric_Pad1.18x1.45mm_HandSolder, B.Cu at (92.1, 71.7)
- added C34: 1uF, Capacitor_SMD:C_0805_2012Metric_Pad1.18x1.45mm_HandSolder, B.Cu at (92.1, 73.8)
- added C35: 100nF, Capacitor_SMD:C_0805_2012Metric_Pad1.18x1.45mm_HandSolder, F.Cu at (92.9, 102.1)
- added C36: 1nF, Capacitor_SMD:C_1210_3225Metric_Pad1.33x2.70mm_HandSolder, F.Cu at (400.6, 105.8)
- added C37: 100nf, Capacitor_SMD:C_1210_3225Metric_Pad1.33x2.70mm_HandSolder, F.Cu at (400.6, 110.0)
- added C38: 10uF, Capacitor_SMD:C_1210_3225Metric_Pad1.33x2.70mm_HandSolder, F.Cu at (400.6, 114.2)
- added C39: 2.2uF, Capacitor_SMD:C_1210_3225Metric_Pad1.33x2.70mm_HandSolder, F.Cu at (400.6, 118.5)
- added C4: 100nF, Capacitor_SMD:C_1210_3225Metric_Pad1.33x2.70mm_HandSolder, F.Cu at (485.4, 98.5)
- added C40: 2.2uF, Capacitor_SMD:C_1210_3225Metric_Pad1.33x2.70mm_HandSolder, F.Cu at (400.6, 122.8)
- added C41: 2.2uF, Capacitor_SMD:C_1210_3225Metric_Pad1.33x2.70mm_HandSolder, F.Cu at (400.6, 127.0)
- added C5: 100nF, Capacitor_SMD:C_1210_3225Metric_Pad1.33x2.70mm_HandSolder, F.Cu at (485.4, 102.8)
- added C6: 100nF, Capacitor_SMD:C_1210_3225Metric_Pad1.33x2.70mm_HandSolder, B.Cu at (79.7, 51.7)
- added C7: 100nF, Capacitor_SMD:C_1210_3225Metric_Pad1.33x2.70mm_HandSolder, F.Cu at (491.4, 90.0)
- added C8: 100nF, Capacitor_SMD:C_1210_3225Metric_Pad1.33x2.70mm_HandSolder, F.Cu at (491.4, 94.2)
- added C9: 100nF, Capacitor_SMD:C_1210_3225Metric_Pad1.33x2.70mm_HandSolder, F.Cu at (491.4, 98.5)
- added J10: USB_C_Receptacle_USB2.0_16P, Connector_USB:USB_C_Receptacle_GCT_USB4105-xx-A_16P_TopMnt_Horizontal, F.Cu at (310.4, 37.4)
- added J11: Conn_01x05, TerminalBlock_RND:TerminalBlock_RND_205-00004_1x05_P5.00mm_Horizontal, F.Cu at (186.4, 9.73)
- added J12: HALL INPUT, Connector_PinSocket_2.00mm:PinSocket_1x05_P2.00mm_Vertical, F.Cu at (305.2, 79.5)
- added J13: Conn_01x04, TerminalBlock_RND:TerminalBlock_RND_205-00003_1x04_P5.00mm_Horizontal, F.Cu at (264.7, 38.5)
- added J14: Conn_01x05, Connector_PinSocket_2.54mm:PinSocket_1x05_P2.54mm_Vertical, F.Cu at (101.1, 48.8)
- added J15: PHASE_A, Connector_Wire:SolderWirePad_1x01_SMD_5x10mm, F.Cu at (423.7, 109.4)
- added J16: PHASE_B, Connector_Wire:SolderWirePad_1x01_SMD_5x10mm, F.Cu at (430.3, 109.4)
- added J17: PHASE_C, Connector_Wire:SolderWirePad_1x01_SMD_5x10mm, F.Cu at (436.9, 109.4)
- added J4: 58-8 OUTPUT, TerminalBlock_Ningbo-Kagnex:TerminalBlock_Ningbo-Kagnex_HB9500_1x02_P9.5mm, F.Cu at (466.4, 110.1)
- added J5: Conn_01x03, TerminalBlock_RND:TerminalBlock_RND_205-00002_1x03_P5.00mm_Horizontal, F.Cu at (61.8, 93.8)
- added J6: Conn_01x03, TerminalBlock_RND:TerminalBlock_RND_205-00002_1x03_P5.00mm_Horizontal, F.Cu at (61.8, 110.1)
- added J7: Conn_01x02, TerminalBlock_RND:TerminalBlock_RND_205-00001_1x02_P5.00mm_Horizontal, F.Cu at (61.5, 59.9)
- added J8: Conn_01x02, TerminalBlock_RND:TerminalBlock_RND_205-00001_1x02_P5.00mm_Horizontal, F.Cu at (61.6, 71.1)
- added J9: Conn_01x02, TerminalBlock_RND:TerminalBlock_RND_205-00001_1x02_P5.00mm_Horizontal, F.Cu at (61.8, 82.4)
- added NT1: NetTie_2, NetTie:NetTie-2_SMD_Pad2.0mm, F.Cu at (497.4, 118.0)
- added Q1: SS8050, Package_TO_SOT_SMD:SOT-23, F.Cu at (422.9, 117.5)
- added Q10: SS8550, Package_TO_SOT_SMD:SOT-23, F.Cu at (437.6, 117.5)
- added Q11: SS8050, Package_TO_SOT_SMD:SOT-23, F.Cu at (437.6, 121.9)
- added Q12: SS8550, Package_TO_SOT_SMD:SOT-23, F.Cu at (437.6, 126.3)
- added Q17: IAUS300N08S5N014TATMA13, IAUS300N08S5N014TATMA1:IAUS300N08S5N014TATMA1, F.Cu at (381.4, 86.4)
- added Q18: IAUS300N08S5N014TATMA13, IAUS300N08S5N014TATMA1:IAUS300N08S5N014TATMA1, F.Cu at (394.5, 86.4)
- added Q19: IAUS300N08S5N014TATMA13, IAUS300N08S5N014TATMA1:IAUS300N08S5N014TATMA1, F.Cu at (407.7, 86.4)
- added Q2: SS8550, Package_TO_SOT_SMD:SOT-23, F.Cu at (422.9, 121.9)
- added Q20: IAUS300N08S5N014TATMA13, IAUS300N08S5N014TATMA1:IAUS300N08S5N014TATMA1, F.Cu at (420.8, 86.4)
- added Q21: IAUS300N08S5N014TATMA13, IAUS300N08S5N014TATMA1:IAUS300N08S5N014TATMA1, F.Cu at (433.9, 86.4)
- added Q22: IAUS300N08S5N014TATMA13, IAUS300N08S5N014TATMA1:IAUS300N08S5N014TATMA1, F.Cu at (447.0, 86.4)
- added Q3: SS8050, Package_TO_SOT_SMD:SOT-23, F.Cu at (422.9, 126.3)
- added Q4: SS8550, Package_TO_SOT_SMD:SOT-23, F.Cu at (427.8, 117.5)
- added Q5: SS8050, Package_TO_SOT_SMD:SOT-23, F.Cu at (427.8, 121.9)
- added Q6: SS8550, Package_TO_SOT_SMD:SOT-23, F.Cu at (427.8, 126.3)
- added Q7: SS8050, Package_TO_SOT_SMD:SOT-23, F.Cu at (432.7, 117.5)
- added Q8: SS8550, Package_TO_SOT_SMD:SOT-23, F.Cu at (432.7, 121.9)
- added Q9: SS8050, Package_TO_SOT_SMD:SOT-23, F.Cu at (432.7, 126.3)
- added R1: 10K, Resistor_SMD:R_1210_3225Metric, F.Cu at (86.0, 76.2)
- added R10: 4.7K, Resistor_SMD:R_1210_3225Metric, F.Cu at (298.6, 66.9)
- added R11: 10K, Resistor_SMD:R_1210_3225Metric, F.Cu at (87.4, 53.7)
- added R12: 10K, Resistor_SMD:R_1210_3225Metric, F.Cu at (87.4, 100.5)
- added R13: 10K, Resistor_SMD:R_1210_3225Metric, F.Cu at (304.2, 54.3)
- added R14: 10K, Resistor_SMD:R_1210_3225Metric, F.Cu at (304.2, 58.5)
- added R15: 10K, Resistor_SMD:R_1210_3225Metric, F.Cu at (304.2, 62.7)
- added R16: 75K, Resistor_SMD:R_1210_3225Metric, F.Cu at (406.4, 105.7)
- added R17: 1K, Resistor_SMD:R_1210_3225Metric, F.Cu at (406.4, 109.9)
- added R18: 10K, Resistor_SMD:R_1210_3225Metric, F.Cu at (406.4, 114.2)
- added R19: 1mR, Resistor_SMD:R_1210_3225Metric, F.Cu at (406.4, 118.4)
- added R2: 10K, Resistor_SMD:R_1210_3225Metric, F.Cu at (87.2, 88.3)
- added R20: 2K, Resistor_SMD:R_1210_3225Metric, F.Cu at (406.4, 122.6)
- added R21: 10R, Resistor_SMD:R_1210_3225Metric, F.Cu at (406.4, 126.8)
- added R22: 10R, Resistor_SMD:R_1210_3225Metric, F.Cu at (412.0, 105.7)
- added R23: 10R, Resistor_SMD:R_1210_3225Metric, F.Cu at (412.0, 109.9)
- added R24: 10R, Resistor_SMD:R_1210_3225Metric, F.Cu at (412.0, 114.2)
- added R25: 10R, Resistor_SMD:R_1210_3225Metric, F.Cu at (412.0, 118.4)
- added R26: 10R, Resistor_SMD:R_1210_3225Metric, F.Cu at (412.0, 122.6)
- added R27: 10K, Resistor_SMD:R_1210_3225Metric, F.Cu at (412.0, 126.8)
- added R28: 10K, Resistor_SMD:R_1210_3225Metric, F.Cu at (417.6, 105.7)
- added R29: 10K, Resistor_SMD:R_1210_3225Metric, F.Cu at (417.6, 109.9)
- added R3: 10K, Resistor_SMD:R_1210_3225Metric, F.Cu at (87.2, 92.5)
- added R4: 10K, Resistor_SMD:R_1210_3225Metric, F.Cu at (87.2, 96.7)
- added R5: 2.2K, Resistor_SMD:R_1210_3225Metric, F.Cu at (293.0, 71.1)
- added R6: 2.2K, Resistor_SMD:R_1210_3225Metric, F.Cu at (293.0, 75.3)
- added R7: 2.2K, Resistor_SMD:R_1210_3225Metric, F.Cu at (298.6, 54.3)
- added R8: 4.7K, Resistor_SMD:R_1210_3225Metric, F.Cu at (298.6, 58.5)
- added R9: 4.7K, Resistor_SMD:R_1210_3225Metric, F.Cu at (298.6, 62.7)
- added U10: IR2130, Package_DIP:DIP-28_W15.24mm, F.Cu at (380.8, 105.7)
- added U3: XC6206PxxxMR, Package_TO_SOT_SMD:SOT-23-3, F.Cu at (503.0, 90.3)
- added U4: LM7805, Package_TO_SOT_THT:TO-220-3_Vertical, F.Cu at (485.6, 114.8)
- added U5: XC6206PxxxMR, Package_TO_SOT_SMD:SOT-23-3, F.Cu at (503.0, 94.8)
- added U6: XC6206PxxxMR, Package_TO_SOT_SMD:SOT-23-3, F.Cu at (503.0, 99.2)
- added U7: LM7805, Package_TO_SOT_THT:TO-220-3_Vertical, F.Cu at (485.6, 120.7)
- added U8: TJA1051T, Package_SO:SOIC-8_3.9x4.9mm_P1.27mm, F.Cu at (308.8, 45.4)
- added U9: STM32G474VETx, Package_QFP:LQFP-100_14x14mm_P0.5mm, F.Cu at (90.8, 64.9)
- added Y1: 8MHz, Crystal:Crystal_HC18-U_Vertical, F.Cu at (77.6, 67.2)
- D1, D2, D3: value D -> U1SM
- J1: value PHASE_B -> Conn_01x02; footprint Connector_Wire:SolderWirePad_1x01_SMD_5x10mm -> TerminalBlock_RND:TerminalBlock_RND_205-00001_1x02_P5.00mm_Horizontal
- J2: value PHASE_A -> +VDC
- J3: value PHASE_C -> -VDC
- R30, R31, R32: value 10R -> 10K
- R33: value 10R -> 10k; footprint Resistor_SMD:R_1210_3225Metric -> Resistor_SMD:R_0805_2012Metric_Pad1.20x1.40mm_HandSolder
- U1: value STM32G474VETx -> LM7805; footprint Package_QFP:LQFP-100_14x14mm_P0.5mm -> Package_TO_SOT_THT:TO-220-3_Vertical
- U2: value IR2133 -> XC6206PxxxMR; footprint Package_DIP:DIP-28_W15.24mm -> Package_TO_SOT_SMD:SOT-23-3; moved to B.Cu
- moved U1 480.6 mm to (485.6, 108.8)
- moved J2 478.5 mm to (497.2, 110.7)
- moved J3 478.5 mm to (503.8, 110.7)
- moved J1 451.0 mm to (466.4, 90.0)
- moved D1 432.0 mm to (445.1, 117.5)
- moved D2 432.0 mm to (445.1, 122.0)
- moved D3 432.0 mm to (445.1, 126.6)
- moved R30 412.6 mm to (417.6, 114.2)
- moved R31 412.6 mm to (417.6, 118.4)
- moved R32 412.6 mm to (417.6, 122.6)
- moved U2 96.3 mm to (83.1, 52.0), turned to 90 degrees
- moved R33 90.8 mm to (102.1, 51.5), turned to 180 degrees
Connections:
- D1 pad 1: /FET_DRIVER/D3 -> /FET_DRIVER/D1
- D2 pad 2: Net-(D2-A) -> +12V
- D3 pad 1: /FET_DRIVER/D1 -> /FET_DRIVER/D3
- J1 pad 1: /FET_DRIVER/VS3 -> +12V
- J2 pad 1: /FET_DRIVER/VS1 -> +VDC
- J3 pad 1: /FET_DRIVER/VS3 -> -VDC
- R30 pad 1: unconnected-(R30-Pad1) -> /FET_DRIVER/VS2
- R31 pad 1: unconnected-(R31-Pad1) -> Net-(Q17-Pad8)
- R31 pad 2: Net-(Q3-Pad1) -> /FET_DRIVER/VS3
- R32 pad 1: unconnected-(R32-Pad1) -> Net-(Q18-Pad8)
- R32 pad 2: Net-(Q2-Pad1) -> /FET_DRIVER/MOS_NEG
- R33 pad 1: unconnected-(R33-Pad1) -> +3V3
- R33 pad 2: Net-(Q4-Pad1) -> /mcu/NRST
- U1 pad 1: unconnected-(U1-PE2-Pad1) -> +12V
- U1 pad 2: unconnected-(U1-PE3-Pad2) -> GND
- U1 pad 3: unconnected-(U1-PE4-Pad3) -> +5V
- U2 pad 1: Net-(D2-A) -> GND
- U2 pad 2: unconnected-(U2-~{HIN1}-Pad2) -> +3V3
- U2 pad 3: unconnected-(U2-~{HIN2}-Pad3) -> +5V
Routing:
- net /mcu/NRST: track 0.00 -> 32.3 mm
- net +3V3: track 0.00 -> 25.7 mm, vias 0 -> 9
- net GND: track 0.00 -> 17.8 mm, vias 0 -> 8
- net /mcu/SVCLK: track 0.00 -> 11.6 mm
- net /mcu/SVDIO: track 0.00 -> 9.08 mm
- net Net-(U9-PF1): track 0.00 -> 6.86 mm
- net /mcu/ADC3_Regen: track 0.00 -> 6.81 mm
- net Net-(U9-PF0): track 0.00 -> 6.77 mm
- net /mcu/GPIO_BRAKE: track 0.00 -> 6.21 mm
- net /mcu/HALT: track 0.00 -> 5.28 mm
- net /mcu/Brake Lights: track 0.00 -> 4.08 mm
- net /mcu/ADC3_ACCELERATOR: track 0.00 -> 3.52 mm
- net Net-(U9-PB8): track 0.00 -> 2.08 mm
- added copper zone on B.Cu, net +3V3
- added copper zone on In1.Cu, net GND
- added copper zone on In2.Cu, net GND
Other:
- copper layers 2 -> 4

Commit message: pcb geçiş v2
Parts:
- added G***: LOGO, LOGO, F.Cu at (55.6, 58.0)
- R1, R11, R12, R13, R14, R15, R2, R21, R3, R4: footprint Resistor_SMD:R_1210_3225Metric -> Resistor_SMD:R_0805_2012Metric_Pad1.20x1.40mm_HandSolder
- moved J12 218.8 mm to (95.3, 17.7), turned to -90 degrees
- moved R8 212.5 mm to (89.5, 21.0)
- moved J11 209.3 mm to (-18.6, 51.9)
- moved R9 208.3 mm to (94.5, 21.0), turned to 180 degrees
- moved R5 207.5 mm to (90.3, 27.1), turned to 90 degrees
- moved R6 205.3 mm to (93.5, 27.1), turned to 90 degrees
- moved R10 204.3 mm to (99.5, 21.0), turned to 180 degrees
- moved R7 203.7 mm to (96.7, 27.1), turned to 90 degrees
- moved C21 150.0 mm to (90.3, 32.1), turned to -90 degrees
- moved C22 147.5 mm to (93.5, 32.1), turned to -90 degrees
- moved C23 145.1 mm to (96.8, 32.1), turned to -90 degrees
- moved J6 93.7 mm to (33.0, 21.0), turned to 180 degrees
- moved J5 76.0 mm to (82.7, 20.7), turned to 180 degrees
- moved C15 64.1 mm to (48.8, 43.6), turned to 90 degrees
- moved C35 63.7 mm to (66.1, 44.3), turned to 90 degrees
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Connections:
- C15 pad 2: Net-(J6-Pin_2) -> /mcu/ADC3_Regen
Routing:
- net /mcu/HALL_A: track 0.00 -> 40.0 mm, vias 0 -> 2
- net /mcu/HALL_B: track 0.00 -> 37.2 mm, vias 0 -> 2
- net Net-(J6-Pin_2): track 0.00 -> 34.4 mm
- net /mcu/HALL_C: track 0.00 -> 31.9 mm, vias 0 -> 2
- net Net-(J5-Pin_2): track 0.00 -> 25.0 mm
- net Net-(J7-Pin_1): track 0.00 -> 24.5 mm
- net /mcu/ADC3_Regen: track 6.81 -> 29.1 mm
- net Net-(J8-Pin_1): track 0.00 -> 22.1 mm
- net Net-(J9-Pin_1): track 0.00 -> 21.7 mm
- net /mcu/GPIO_BRAKE: track 6.21 -> 23.8 mm
- net /mcu/HALT: track 5.28 -> 19.1 mm
- net GND: track 17.8 -> 29.3 mm, vias 8 -> 11
- net Net-(J12-Pin_1): track 0.00 -> 10.2 mm
- net /mcu/Brake Lights: track 4.08 -> 12.5 mm
- net Net-(J12-Pin_3): track 0.00 -> 8.40 mm
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
Commit message: pcb geçiş v2
Parts:
- removed C10, C11, C12, C4, C5, C7, C8, C9: 100nF, Capacitor_SMD:C_1210_3225Metric_Pad1.33x2.70mm_HandSolder
- removed C36: 1nF, Capacitor_SMD:C_1210_3225Metric_Pad1.33x2.70mm_HandSolder
- removed J11: Conn_01x05, TerminalBlock_RND:TerminalBlock_RND_205-00004_1x05_P5.00mm_Horizontal
- removed Q1, Q11, Q3, Q5, Q7, Q9: SS8050, Package_TO_SOT_SMD:SOT-23
- removed Q10, Q12, Q2, Q4, Q6, Q8: SS8550, Package_TO_SOT_SMD:SOT-23
- removed Q17, Q18: IAUS300N08S5N014TATMA13, IAUS300N08S5N014TATMA1:IAUS300N08S5N014TATMA1
- removed R28, R29, R30, R31, R32: 10K, Resistor_SMD:R_1210_3225Metric
- removed U3: XC6206PxxxMR, Package_TO_SOT_SMD:SOT-23-3
- removed U4: LM7805, Package_TO_SOT_THT:TO-220-3_Vertical
- added C42: 1nF, Capacitor_SMD:C_1210_3225Metric_Pad1.33x2.70mm_HandSolder, B.Cu at (73.5, 76.3)
- added Q23: IAUS300N08S5N014TATMA13, IAUS300N08S5N014TATMA1:IAUS300N08S5N014TATMA, F.Cu at (8.26, 115.2)
- added Q24: IAUS300N08S5N014TATMA13, IAUS300N08S5N014TATMA1:IAUS300N08S5N014TATMA, F.Cu at (30.2, 115.2)
- added U11: TC4422, Package_DIP:DIP-8_W7.62mm, F.Cu at (13.6, 99.9)
- added U12: TC4422, Package_DIP:DIP-8_W7.62mm, F.Cu at (125.9, 99.4)
- added U13: TC4422, Package_DIP:DIP-8_W7.62mm, F.Cu at (81.5, 100.0)
- added U14: TC4422, Package_DIP:DIP-8_W7.62mm, F.Cu at (35.6, 100.0)
- C37, C38: moved to B.Cu
- J13: footprint TerminalBlock_RND:TerminalBlock_RND_205-00003_1x04_P5.00mm_Horizontal -> Connector_PinHeader_2.54mm:PinHeader_1x04_P2.54mm_Vertical
- J4: value 58-8 OUTPUT -> Conn_01x02; footprint TerminalBlock_Ningbo-Kagnex:TerminalBlock_Ningbo-Kagnex_HB9500_1x02_P9.5mm -> TerminalBlock_RND:TerminalBlock_RND_205-00001_1x02_P5.00mm_Horizontal
- R16: value 75K -> 22K
- R19: value 1mR -> 10mR; footprint Resistor_SMD:R_1210_3225Metric -> Resistor_SMD:R_Shunt_Vishay_WSR2_WSR3_KelvinConnection
- R21: footprint Resistor_SMD:R_0805_2012Metric_Pad1.20x1.40mm_HandSolder -> Resistor_SMD:R_1210_3225Metric_Pad1.30x2.65mm_HandSolder
- R27: footprint Resistor_SMD:R_1210_3225Metric -> Resistor_SMD:R_0805_2012Metric_Pad1.20x1.40mm_HandSolder
- U5, U6: value XC6206PxxxMR -> TC4422; footprint Package_TO_SOT_SMD:SOT-23-3 -> Package_DIP:DIP-8_W7.62mm
- moved J2 498.7 mm to (0.50, 66.2), turned to 90 degrees
- moved NT1 476.1 mm to (23.5, 73.0), turned to -90 degrees
- moved J3 473.0 mm to (31.4, 86.1)
- moved J4 456.2 mm to (12.1, 68.2), turned to 90 degrees
- moved U6 443.7 mm to (59.3, 99.9), turned to -90 degrees
- moved J17 416.3 mm to (20.8, 123.2), turned to -90 degrees
- moved U5 398.8 mm to (104.2, 99.4), turned to -90 degrees
- moved C14 396.0 mm to (106.0, 38.5)
- moved R25 395.1 mm to (17.0, 107.2), turned to -90 degrees
- moved C13 391.3 mm to (109.0, 46.8), turned to 180 degrees
- moved C2 386.8 mm to (105.5, 17.1)
- moved U1 385.3 mm to (110.6, 20.4), turned to 180 degrees
- moved U7 383.6 mm to (110.2, 41.8), turned to 180 degrees
- moved C1 381.0 mm to (110.7, 17.1), turned to 180 degrees
- moved Q22 378.1 mm to (70.3, 118.9), turned to 90 degrees
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Connections:
- C37 pad 2: -VDC -> Net-(C37-Pad2)
- C38 pad 2: -VDC -> Net-(C37-Pad2)
- D1 pad 2: Net-(D1-A) -> +12V
- D3 pad 2: Net-(D1-A) -> +12V
- J10 pad A4: Net-(J10-VBUS-PadA4) -> +5V
- J10 pad A9: Net-(J10-VBUS-PadA4) -> +5V
- J10 pad B4: Net-(J10-VBUS-PadA4) -> +5V
- J10 pad B9: Net-(J10-VBUS-PadA4) -> +5V
- Q19 pad 8: /FET_DRIVER/VS1 -> Net-(Q19-Pad8)
- Q20 pad 8: /FET_DRIVER/VS2 -> Net-(Q20-Pad8)
- Q21 pad 8: /FET_DRIVER/MOS_NEG -> Net-(Q21-Pad8)
- Q22 pad 8: /FET_DRIVER/MOS_NEG -> Net-(Q22-Pad8)
- R16 pad 1: unconnected-(R16-Pad1) -> Net-(U10-CA-)
- R16 pad 2: unconnected-(R16-Pad2) -> /FET_DRIVER/CA0
- R19 pad 2: /FET_DRIVER/MOS_NEG -> -VDC
- R20 pad 1: /FET_DRIVER/MOS_NEG -> Net-(U10-VS0)
- R27 pad 1: Net-(Q22-Pad8) -> Net-(U8-CANH)
- R27 pad 2: /FET_DRIVER/MOS_NEG -> Net-(U8-CANL)
- U10 pad 13: /FET_DRIVER/MOS_NEG -> Net-(U10-VS0)
- U10 pad 14: /FET_DRIVER/LOT3 -> Net-(U10-LO3)
- U10 pad 15: /FET_DRIVER/LOT2 -> Net-(U10-LO2)
- U10 pad 16: /FET_DRIVER/LOT1 -> Net-(U10-LO1)
- U10 pad 19: /FET_DRIVER/HOT3 -> Net-(U10-HO3)
- U10 pad 23: /FET_DRIVER/HOT2 -> Net-(U10-HO2)
- U10 pad 27: /FET_DRIVER/HOT1 -> Net-(U10-HO1)
- U5 pad 1: GND -> +12V
- U5 pad 2: +3.3VA -> Net-(U10-HO1)
- U5 pad 3: +5V -> unconnected-(U5-NC-Pad3)
- U6 pad 1: GND -> +12V
- U6 pad 2: +5V -> Net-(U10-HO2)
- U6 pad 3: +5V -> unconnected-(U6-NC-Pad3)
- U8 pad 3: unconnected-(U8-VCC-Pad3) -> +5V
- U8 pad 4: unconnected-(U8-RXD-Pad4) -> /mcu/CAN_TX
- U9 pad 27: /mcu/SPICLK -> unconnected-(U9-PA5-Pad27)
- U9 pad 28: /mcu/MISO -> unconnected-(U9-PA6-Pad28)
- U9 pad 29: /mcu/MOSI -> unconnected-(U9-PA7-Pad29)
Routing:
- net +12V: track 0.00 -> 152.6 mm, vias 0 -> 46
- net -VDC: track 0.00 -> 106.3 mm, vias 0 -> 1
- net Net-(U10-HO3): track 0.00 -> 73.7 mm
- net /FET_DRIVER/VS3: track 0.00 -> 66.1 mm, vias 0 -> 31
- net Net-(U10-LO1): track 0.00 -> 65.3 mm
- net /FET_DRIVER/VS2: track 0.00 -> 44.8 mm, vias 0 -> 31
- net /FET_DRIVER/VS1: track 0.00 -> 43.4 mm, vias 0 -> 31
- net Net-(U10-LO3): track 0.00 -> 42.7 mm
- net Net-(U10-HO2): track 0.00 -> 38.0 mm
- net Net-(U10-ITRIP): track 0.00 -> 37.8 mm
- net /FET_DRIVER/CA0: track 0.00 -> 30.8 mm, vias 0 -> 2
- net Net-(U10-VS0): track 0.00 -> 29.4 mm, vias 0 -> 1
- net +5V: track 4.59 -> 33.0 mm, vias 0 -> 3
- net Net-(J13-Pin_2): track 0.00 -> 25.9 mm
- net Net-(J13-Pin_3): track 0.00 -> 25.7 mm
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- added copper zone on In2.Cu, net +12V
- added copper zone on F.Cu, net +5V
- added copper zone on F.Cu, net +VDC
- added copper zone on F.Cu, net -VDC
- added copper zone on F.Cu, net /FET_DRIVER/MOS_NEG
- added copper zone on In1.Cu, net /FET_DRIVER/MOS_NEG
- added copper zone on In2.Cu, net /FET_DRIVER/MOS_NEG
- added copper zone on F.Cu, net /FET_DRIVER/VS1
- added copper zone on F.Cu, net /FET_DRIVER/VS2
- added copper zone on F.Cu, net /FET_DRIVER/VS3
- added copper zone on F.Cu, net Net-(U10-VS0)
Other:
- board outline added: 142.2 x 124.5 mm
- board text added: "SEM"

Commit message: pcb geçiş v2
Parts:
- added C10: 4.7uF, Capacitor_SMD:C_1210_3225Metric_Pad1.33x2.70mm_HandSolder, B.Cu at (33.3, 63.1)
- added C36: 100nF, Capacitor_SMD:C_1210_3225Metric_Pad1.33x2.70mm_HandSolder, B.Cu at (77.4, 93.6)
- added C4: 680uF, Capacitor_THT:CP_Radial_D10.0mm_P5.00mm, F.Cu at (116.2, 20.7)
- added C43: 100nF, Capacitor_SMD:C_1210_3225Metric_Pad1.33x2.70mm_HandSolder, B.Cu at (102.0, 93.7)
- added C44: 100nF, Capacitor_SMD:C_1210_3225Metric_Pad1.33x2.70mm_HandSolder, B.Cu at (123.3, 93.5)
- added C45: 100nF, Capacitor_SMD:C_1210_3225Metric_Pad1.33x2.70mm_HandSolder, B.Cu at (12.0, 100.2)
- added C46: 100nF, Capacitor_SMD:C_1210_3225Metric_Pad1.33x2.70mm_HandSolder, B.Cu at (55.7, 99.9)
- added C47: 100nF, Capacitor_SMD:C_1210_3225Metric_Pad1.33x2.70mm_HandSolder, B.Cu at (102.0, 100.0)
- added C48: 10uF, Capacitor_SMD:C_1210_3225Metric_Pad1.33x2.70mm_HandSolder, B.Cu at (33.9, 99.9)
- added C49: 10uF, Capacitor_SMD:C_1210_3225Metric_Pad1.33x2.70mm_HandSolder, B.Cu at (77.3, 99.9)
- added C5: 680uF, Capacitor_THT:CP_Radial_D10.0mm_P5.00mm, F.Cu at (116.4, 31.3)
- added C50: 10uF, Capacitor_SMD:C_1210_3225Metric_Pad1.33x2.70mm_HandSolder, B.Cu at (123.1, 99.8)
- added C51: 100nF, Capacitor_SMD:C_1210_3225Metric_Pad1.33x2.70mm_HandSolder, B.Cu at (55.9, 93.5)
- added C52: 100nF, Capacitor_SMD:C_1210_3225Metric_Pad1.33x2.70mm_HandSolder, B.Cu at (12.2, 93.6)
- added C53: 100nF, Capacitor_SMD:C_1210_3225Metric_Pad1.33x2.70mm_HandSolder, B.Cu at (33.9, 93.7)
- added C7: 1000uF / 100V, Capacitor_THT:CP_Radial_D18.0mm_P7.50mm, F.Cu at (40.3, 59.3)
- added C8: 1000uF 100V, Capacitor_THT:CP_Radial_D18.0mm_P7.50mm, F.Cu at (21.7, 59.6)
- added C9: 4.7uF, Capacitor_SMD:C_1210_3225Metric_Pad1.33x2.70mm_HandSolder, B.Cu at (29.9, 63.1)
- C39, C40, C41: value 2.2uF -> 10uF
- G***, R16, R17, R18, R20: moved to B.Cu
- Q19, Q20, Q21, Q22: footprint IAUS300N08S5N014TATMA1:IAUS300N08S5N014TATMA1 -> IAUS300N08S5N014TATMA1:IAUS300N08S5N014TATMA
- moved NT1 88.3 mm to (111.7, 69.2)
- moved J3 81.4 mm to (111.7, 72.5), turned to 90 degrees
- moved G*** 31.6 mm to (59.2, 46.4), turned to 180 degrees
- moved R20 31.1 mm to (75.0, 73.0), turned to 180 degrees
- moved R18 25.8 mm to (70.3, 73.0), turned to 180 degrees
- moved J4 25.3 mm to (27.4, 48.0), turned to 180 degrees
- moved R19 17.3 mm to (58.5, 75.6), turned to -90 degrees
- moved J2 16.4 mm to (11.9, 78.0)
- moved R17 14.9 mm to (69.2, 64.0), turned to -90 degrees
- moved J6 10.3 mm to (38.7, 29.6), turned to -90 degrees
- moved Q19 10.0 mm to (100.4, 111.7)
- moved Q21 9.68 mm to (121.8, 111.7)
- moved Q20 9.43 mm to (54.4, 111.6)
- moved Q22 9.14 mm to (75.8, 111.6)
- moved Q23 4.52 mm to (11.1, 111.7)
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Routing:
- net +12V: track 152.6 -> 378.9 mm, vias 46 -> 3
- net Net-(U10-ITRIP): track 37.8 -> 9.56 mm
- net -VDC: track 106.3 -> 125.7 mm, vias 1 -> 126
- net +VDC: track 16.9 -> 35.6 mm, vias 0 -> 622
- net Net-(J6-Pin_2): track 34.4 -> 15.8 mm
- net Net-(U10-LO1): track 65.3 -> 78.0 mm
- net GND: track 53.4 -> 63.9 mm, vias 34 -> 69
- net Net-(U10-CA-): track 16.8 -> 7.20 mm
- net /FET_DRIVER/VS2: track 44.8 -> 39.2 mm, vias 31 -> 51
- net /FET_DRIVER/VS3: track 66.1 -> 71.2 mm, vias 31 -> 53
- net /FET_DRIVER/CA0: track 30.8 -> 25.7 mm, vias 2 -> 1
- net Net-(U10-VS0): track 29.4 -> 26.5 mm
- net /FET_DRIVER/FAULT: track 14.9 -> 12.2 mm
- net Net-(U10-HO3): track 73.7 -> 71.5 mm
- net /FET_DRIVER/D1: track 11.8 -> 9.84 mm
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- added copper zone on In1.Cu, net +VDC
- added copper zone on In2.Cu, net +VDC
- added copper zone on B.Cu, net -VDC
- added copper zone on In1.Cu, net -VDC
- added copper zone on In2.Cu, net -VDC
- added copper zone on B.Cu, net /FET_DRIVER/MOS_NEG
- added copper zone on B.Cu, net /FET_DRIVER/VS1
- added copper zone on In1.Cu, net /FET_DRIVER/VS1
- added copper zone on In2.Cu, net /FET_DRIVER/VS1
- added copper zone on B.Cu, net /FET_DRIVER/VS2
- added copper zone on In1.Cu, net /FET_DRIVER/VS2
- added copper zone on In2.Cu, net /FET_DRIVER/VS2
- added copper zone on B.Cu, net /FET_DRIVER/VS3
- added copper zone on In1.Cu, net /FET_DRIVER/VS3
- added copper zone on In2.Cu, net /FET_DRIVER/VS3
- added copper zone on F.Cu, net GND
- removed copper zone on In2.Cu, net +12V
- removed copper zone on F.Cu, net Net-(U10-VS0)
Other:
- board outline removed

Commit message: pcb geçiş v2
Parts:
- added G***: LOGO, LOGO, F.Cu at (19.4, 87.7)
- added G***: LOGO, LOGO, B.Cu at (19.4, 76.7)
- G***: moved to F.Cu
- moved G*** 50.2 mm to (11.1, 32.2), turned to 0 degrees
- moved J2 8.37 mm to (7.00, 71.2)
- moved R19 0.57 mm to (57.9, 75.5)
- moved C42 0.38 mm to (69.0, 77.1)
Routing:
- net /mcu/NRST: track 29.7 -> 27.3 mm
- net GND: track 63.9 -> 64.9 mm, vias 69 -> 66
- net Net-(U10-VS0): track 26.5 -> 27.5 mm
- net -VDC: vias 126 -> 156
- added copper zone on B.Cu, net +VDC
Other:
- board outline added: 132.5 x 118.2 mm
- board text added: "5v"
- board text added: "A"
- board text added: "Accel"
- board text added: "B"
- board text added: "Brake"
- board text added: "Brake-Lights"
- board text added: "C"
- board text added: "GND"
- board text added: "HALT"
- board text added: "REGEN"
